File: hardware/mini_r2_0/cad/HM_Nightfall-mini-2e_v1.brd (EAGLE design)
At the start: 39 x 70 mm, 86 parts, among them K1 62201021121, Q2 IRLML6402TRPBF, U1 AP2210N-3.3TRG1, U2 MP6551GQB-P, U3 MP6551GQB-P, U4 ISM330DHCXTR, U5 STM32F413CHU6TRUFQFPN-48_7X7X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, U6 CY15B108QI-20LPXC

Commit message: Update mini CAD files
Routing:
- net GND: vias 55 -> 56
Changed lines of the file:
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@@
 <wire x1="-0.254" y1="-5.207" x2="-0.254" y2="-6.35" width="0.508" layer="16"/>
 <wire x1="-1.27" y1="-4.191" x2="-0.254" y2="-5.207" width="0.508" layer="16"/>
+<via x="6.477" y="-1.905" extent="1-16" drill="0.3"/>
 </signal>
 <signal name="SENSOR_FR">
@@
 <wire x1="-18.0364" y1="-13.9619625" x2="-18.4069625" y2="-13.5914" width="0.254" layer="16"/>
 <wire x1="-18.4069625" y1="-13.5914" x2="-18.9310375" y2="-13.5914" width="0.254" layer="16"/>
-<wire x1="-18.9310375" y1="-13.5914" x2="-19.257775" y2="-13.9181375" width="0.254" layer="16"/>
 <wire x1="-11.43" y1="-19.304" x2="-15.78853125" y2="-19.304" width="0.254" layer="16"/>
 <wire x1="-15.78853125" y1="-19.304" x2="-18.0364" y2="-17.05613125" width="0.254" layer="16"/>
@@
 <wire x1="12.573" y1="8.001" x2="11.97136875" y2="8.60263125" width="0.254" layer="1"/>
 </signal>
-<signal name="N$14">
-<via x="6.477" y="-1.905" extent="1-16" drill="0.3"/>
-</signal>
 </signals>
